File: Gameduino.brd (EAGLE design)
At the start: 68.6 x 53.3 mm, 11 parts

Commit message: Add files via upload
Parts:
- added R1, R2, R4, R6, R7: 10k‎Ω, AUTODESK_CIRCUITS_BREADBOARD:0207/10
Connections:
- removed net N$11 (its old number): S1.1, U5.8
- new net N$12: R1.2, S5.3
- new net N$13: R2.2, S2.3
- new net N$14: R4.2, S3.3
- new net N$15: R6.2, S4.3
- new net N$16: S5.4, U5.A5
- new net N$17: S6.4, U5.A0
- new net N$18: R7.2, S6.3
- new net N$19: S1.4, U5.A1
- new net N$20: S4.4, U5.A2
- new net N$21: S3.4, U5.A3
- new net N$22: S2.4, U5.A4
- net N$1: now also R1.1, R2.1, R4.1, R6.1, R7.1
- net N$10: no longer S1.4
