File: Gameduino 2 Player.brd (EAGLE design)
At the start: 68.6 x 53.3 mm, 14 parts

Commit message: Add files via upload
Parts:
- added R10, R11, R12, R2, R4, R6, R7, R8, R9: 10k‎Ω, AUTODESK_CIRCUITS_BREADBOARD:0207/10
- added S10, S11, S6, S7, S8, S9: (no value), AUTODESK_CIRCUITS_BREADBOARD:TL1105
- moved R5 88.9 mm to (5.00, 213.3)
- moved S2 12.7 mm to (5.00, 124.4)
Connections:
- removed net N$19 (its old number): R3.1, Rpot3.A, S1.4, U5.5V, U6.2
- removed net N$20 (its old number): R5.2, S1.3
- new net N$22: R2.2, S2.3
- new net N$23: S2.4, U1.A0, U5.A0
- new net N$24: S1.4, U1.RESET, U5.RESET
- new net N$25: R4.2, S3.3
- new net N$26: R5.2, S4.3
- new net N$27: R6.2, S6.3
- new net N$28: R8.2, S5.3
- new net N$29: S7.4, U1.A5
- new net N$30: S8.4, U1.A4
- new net N$31: S10.4, U1.A3
- new net N$32: S9.4, U1.A2
- new net N$33: S3.4, U5.A5
- new net N$34: S4.4, U5.A4
- new net N$35: S5.4, U5.A3
- new net N$36: S6.4, U5.A2
- new net N$37: S11.4, U1.A1, U5.A1
- net N$1: now also R10.1, R11.1, R12.1, R2.1, R4.1, R6.1, R7.1, R8.1, R9.1, S1.3
- net N$21: now also R3.1, Rpot3.A, U5.5V, U6.2; no longer S1.1, U1.8, U5.8
